File: Schematics/TransmitterTiny/board.sch (EAGLE design)
At the start: 12 parts, among them IC1 TINY13-20PU, T1 2N2222

Commit message: Finished board
Parts:
- C3: device SparkFun-Capacitors:CAPPTH -> SparkFun-Capacitors:CAPPTH1
Changed lines of the file:
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@@
 <part name="C1" library="SparkFun-Capacitors" deviceset="CAP" device="PTH"/>
 <part name="C2" library="SparkFun-Capacitors" deviceset="CAP" device="PTH"/>
-<part name="C3" library="SparkFun-Capacitors" deviceset="CAP" device="PTH"/>
+<part name="C3" library="SparkFun-Capacitors" deviceset="CAP" device="PTH1"/>
 <part name="L1" library="SparkFun-Passives" deviceset="INDUCTOR" device="AXIAL-0.6"/>
 <part name="T1" library="adafruit" deviceset="2N2222" device=""/>
@@
 </segment>
 </net>
-<net name="N$10" class="0">
+<net name="N$2" class="0">
 <segment>
 <pinref part="USBSERIAL" gate="1" pin="1"/>
